File: DC-DC.kicad_sch (KiCad schematic)
At the start: 16 parts

Commit message: add digikey symbols
Parts:
- added U5: LMR38020SDDAR, DDA0008E-IPC_A, symbol custom_symbols:LMR38020SDDAR
Connections:
- net +5V0_board: now also C10.1, C7.1, C8.1, C9.1, L1.2, R30.2
- net GND: now also R33.1
- net at R33.2: now also R30.1, U5.5 (FB)
- net at C6.1: now also L1.1, U5.7 (BOOT)
- net at C6.2: now also U5.8 (SW)
Other:
- moved on the sheet: C6, L1, R30, R33
