File: MCU.kicad_sch (KiCad schematic)
At the start: 28 parts, among them J4 Conn_01x12_MountingPin, Q2 MMBT3904, Q3 MMBT3904, SW1 SW_DPDT_x2, SW2 SW_Push, SW3 SW_Push, U1 ESP32-C3-WROOM-02, U2 CP2102N-Axx-xQFN28, U3 LIS3DH

Commit message: finish protection sheet
Connections:
- net DTR: no longer Q3.2 (E)
- net RTS: no longer Q2.2 (E)
- net at Q2.1 (B), R11.1: now also Q3.2 (E)
- net at Q3.1 (B), R12.1: now also Q2.2 (E)
Changed lines of the file:
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@@
 	)
 	(junction
-		(at 149.86 181.61)
-		(diameter 0)
-		(color 0 0 0 0)
-	)
-	(junction
 		(at 306.07 129.54)
 		(diameter 0)
@@
 	)
 	(junction
+		(at 161.29 181.61)
+		(diameter 0)
+		(color 0 0 0 0)
+	)
+	(junction
 		(at 97.79 60.96)
 		(diameter 0)
@@
 	)
 	(junction
-		(at 35.56 175.26)
+		(at 162.56 198.12)
 		(diameter 0)
 		(color 0 0 0 0)
 	)
 	(junction
-		(at 146.05 198.12)
+		(at 35.56 175.26)
 		(diameter 0)
 		(color 0 0 0 0)
@@
 	(wire
 		(pts
+			(xy 162.56 187.96) (xy 170.18 187.96)
+		)
+		(stroke
+			(width 0)
+			(type default)
+		)
+	)
+	(wire
+		(pts
 			(xy 370.84 68.58) (xy 367.03 68.58)
 		)
@@
 	(wire
 		(pts
-			(xy 146.05 187.96) (xy 170.18 187.96)
-		)
-		(stroke
-			(width 0)
-			(type default)
-		)
-	)
-	(wire
-		(pts
 			(xy 356.87 50.8) (xy 370.84 50.8)
 		)
@@
 	(wire
 		(pts
-			(xy 146.05 198.12) (xy 135.89 198.12)
+			(xy 135.89 198.12) (xy 152.4 198.12)
 		)
 		(stroke
@@
 	(wire
 		(pts
-			(xy 135.89 181.61) (xy 149.86 181.61)
+			(xy 135.89 181.61) (xy 152.4 181.61)
 		)
 		(stroke
@@
 	(wire
 		(pts
-			(xy 149.86 181.61) (xy 152.4 181.61)
-		)
-		(stroke
-			(width 0)
-			(type default)
-		)
-	)
-	(wire
-		(pts
 			(xy 92.71 162.56) (xy 102.87 162.56)
 		)
@@
 	(wire
 		(pts
-			(xy 149.86 191.77) (xy 149.86 181.61)
-		)
-		(stroke
-			(width 0)
-			(type default)
-		)
-	)
-	(wire
-		(pts
 			(xy 170.18 207.01) (xy 193.04 207.01)
 		)
@@
 	(wire
 		(pts
+			(xy 161.29 181.61) (xy 160.02 181.61)
+		)
+		(stroke
+			(width 0)
+			(type default)
+		)
+	)
+	(wire
+		(pts
 			(xy 80.01 224.79) (xy 80.01 223.52)
 		)
@@
 	(wire
 		(pts
+			(xy 161.29 191.77) (xy 170.18 191.77)
+		)
+		(stroke
+			(width 0)
+			(type default)
+		)
+	)
+	(wire
+		(pts
 			(xy 306.07 149.86) (xy 306.07 172.72)
 		)
@@
 	(wire
 		(pts
-			(xy 146.05 198.12) (xy 152.4 198.12)
+			(xy 113.03 106.68) (xy 143.51 106.68)
 		)
 		(stroke
@@
 	(wire
 		(pts
-			(xy 113.03 106.68) (xy 143.51 106.68)
+			(xy 161.29 191.77) (xy 161.29 181.61)
 		)
 		(stroke
@@
 	(wire
 		(pts
-			(xy 170.18 191.77) (xy 149.86 191.77)
+			(xy 162.56 187.96) (xy 162.56 198.12)
 		)
 		(stroke
@@
 	(wire
 		(pts
-			(xy 146.05 198.12) (xy 146.05 187.96)
-		)
-		(stroke
-			(width 0)
-			(type default)
-		)
-	)
-	(wire
-		(pts
 			(xy 22.86 175.26) (xy 35.56 175.26)
 		)
@@
 	(wire
 		(pts
-			(xy 160.02 181.61) (xy 162.56 181.61)
+			(xy 161.29 181.61) (xy 162.56 181.61)
 		)
 		(stroke
@@
 			"54WE2iG/ZyYWdKtb+tG5Y4V3pmIPAADSS5m5d3Ges9ARAADozqvX2dNuZCbkqd0V3le6L62K9kZA"
 			"0JKROiqW09pAR6zhePzP6h8pvaWJyWKl1Yq1Syn1QUFBQfFS8zfj+8VlA/NmwwAAAABJRU5ErkJg"
-			"gg=="
+			"ggAAAAAAAAAAAAAAAAAAAAAAAAAAAAAAAAAAAAAAAAAAAAAAAAAAAAAAAAAAAAAAAAAAAAAAAAAA"
+			"AAAAAAAAAAAAAAAAAAAAAAAAAAAAAAAAAAAAAAAAAAAAAAAAAAAAAAAAAAAAAAAAAAAAAAAAAAAA"
+			"AAAAAAAAAAAAAAAAAAAAAAAAAAAAAAAAAAAAAAAAAAAAAAAAAAAAAAAAAAAAAAAAAAAAAAAAAAAA"
+			"AAAAAAAAAAAAAAAAAAAAAAAAAAAAAAAAAAAAAAAAAAAAAAAAAAAAAAAAAAAAAAAAAAAAAAAAAAAA"
+			"AAAAAAAAAAAAAAAAAAAAAAAAAAAAAAAAAAAAAAAAAAAAAAAAAAAAAAAAAAAAAAAAAAAAAAAAAAAA"
+			"AAAAAAAAAAAAAAAAAAAAAAAAAAAAAAAAAAAAAAAAAAAAAAAAAAAAAAAAAAAAAAAAAAAAAAAAAAAA"
+			"AAAAAAAAAAAAAAAAAAAAAAAAAAAAAAAAAAAAAAAAAAAAAAAAAAAAAAAAAAAAAAAAAAAAAAAAAAAA"
+			"AAAAAAAAAAAAAAAAAAAAAAAAAAAAAAAAAAAAAAAAAAAAAAAAAAAAAAAAAAAAAAAAAAAAAAAAAAAA"
+			"AAAAAAAAAAAAAAAAAAAAAAAAAAAAAAAAAAAAAAAAAAAAAAAAAAAAAAAAAAAAAAAAAAAAAAAAAAAA"
+			"AAAAAAAAAAAAAAAAAAAAAAAAAAAAAAAAAAAAAAAAAAAAAAAAAAAAAAAAAAAAAAAAAAAAAAAAAAAA"
+			"AAAAAAAAAAAAAAAAAAAAAAAAAAAAAAAAAAAAAAAAAAAAAAAAAAAAAAAAAAAAAAAAAAAAAAAAAAAA"
+			"AAAAAAAAAAAAAAAAAAAAAAAAAAAAAAAAAAAAAAAAAAAAAAAAAAAAAAAAAAAAAAAAAAAAAAAAAAAA"
+			"AAAAAAAAAAAAAAAAAAAAAAAAAAAAAAAAAAAAAAAAAAAAAAAAAAAAAAAAAAAAAAAAAAAAAAAAAAAA"
+			"AAAAAAAAAAAAAAAAAAAAAAAAAAAAAAAAAAAAAAAAAAAAAAAAAAAAAAAAAAAAAAAAAAAAAAAAAAAA"
+			"AAAAAAAAAAAAAAAAAAAAAAAAAAAAAAAAAAAAAAAAAAAAAAAAAAAAAAAAAAAAAAAAAAAAAAAAAAAA"
+			"AAAAAAAAAAAAAAAAAAAAAAAAAAAAAAAAAAAAAAAAAAAAAAAAAAAAAAAAAAAAAAAAAAAAAAAAAAAA"
+			"AAAAAAAAAAAAAAAAAAAAAAAAAAAAAAAAAAAAAAAAAAAAAAAAAAAAAAAAAAAAAAAAAAAAAAAAAAAA"
+			"AAAAAAAAAAAAAAAAAAAAAAAAAAAAAAAAAAAAAAAAAAAAAAAAAAAAAAAAAAAAAAAAAAAAAAAAAAAA"
+			"AAAAAAAAAAAAAAAAAAAAAAAAAAAAAAAAAAAAAAAAAAAAAAAAAAAAAAAAAAAAAAAAAAAAAAAAAAAA"
+			"AAAAAAAAAAAAAAAAAAAAAAAAAAAAAAAAAAAAAAAAAAAAAAAAAAAAAAAAAAAAAAAAAAAAAAAAAAAA"
+			"AAAAAAAAAAAAAAAAAAAAAAAAAAAAAAAAAAAAAAAAAAAAAAAAAAAAAAAAAAAAAAAAAAAAAAAAAAAA"
+			"AAAAAAAAAAAAAAAAAAAAAAAAAAAAAAAAAAAAAAAAAAAAAAAAAAAAAAAAAAAAAAAAAAAAAAAAAAAA"
+			"AAAAAAAAAAAAAAAAAAAAAAAAAAAAAAAAAAAAAAAAAAAAAAAAAAAAAAAAAAAAAAAAAAAAAAAAAAAA"
+			"AAAAAAAAAAAAAAAAAAAAAAAAAAAAAAAAAAAAAAAAAAAAAAAAAAAAAAAAAAAAAAAAAAAAAAAAAAAA"
+			"AAAAAAAAAAAAAAAAAAAAAAAAAAAAAAAAAAAAAAAAAAAAAAAAAAAAAAAAAAAAAAAAAAAAAAAAAAAA"
+			"AAAAAAAAAAAAAAAAAAAAAAAAAAAAAAAAAAAAAAAAAAAAAAAAAAAAAAAAAAAAAAAAAAAAAAAAAAAA"
+			"AAAAAAAAAAAAAAAAAAAAAAAAAAAAAAAAAAAAAAAAAAAAAAAAAAAAAAAAAAAAAAAAAAAAAAAAAAAA"
+			"AAAAAAAAAAAAAAAAAAAAAAAAAAAAAAAAAAAAAAAAAAAAAAAAAAAAAAAAAAAAAAAAAAAAAAAAAAAA"
+			"AAAAAAAAAAAAAAAAAAAAAAAAAAAAAAAAAAAAAAAAAAAAAAAAAAAAAAAAAAAAAAAAAAAAAAAAAAAA"
+			"AAAAAAAAAAAAAAAAAAAAAAAAAAAAAAAAAAAAAAAAAAAAAAAAAAAAAAAAAAAAAAAAAAAAAAAAAAAA"
+			"AAAAAAAAAAAAAAAAAAAAAAAAAAAAAAAAAAAAAAAAAAAAAAAAAAAAAAAAAAAAAAAAAAAAAAAAAAAA"
+			"AAAAAAAAAAAAAAAAAAAAAAAAAAAAAAAAAAAAAAAAAAAAAAAAAAAAAAAAAAAAAAAAAAAAAAAAAAAA"
+			"AAAAAAAAAAAAAAAAAAAAAAAAAAAAAAAAAAAAAAAAAAAAAAAAAAAAAAAAAAAAAAAAAAAAAAAAAAAA"
+			"AAAAAAAAAAAAAAAAAAAAAAAAAAAAAAAAAAAAAAAAAAAAAAAAAAAAAAAAAAAAAAAAAAAAAAAAAAAA"
+			"AAAAAAAAAAAAAAAAAAAAAAAAAAAAAAAAAAAAAAAAAAAAAAAAAAAAAAAAAAAAAAAAAAAAAAAAAAAA"
+			"AAAAAAAAAAAAAAAAAAAAAAAAAAAAAAAAAAAAAAAAAAAAAAAAAAAAAAAAAAAAAAAAAAAAAAAAAAAA"
+			"AA=="
 		)
 	)
@@
 			"AAAAAAAAAAAAAAAAAAAPAAAAAAAAAAC9colxAQAAAAAAAAAAAAAAAAAAAAAAAA8AAAAAAAAAAGl0"
 			"a2EgVGV4dAAAAAAAAAAAAAAAAAAADwAAAAAAAAAAAAAAAAAAAAAAAAAAAAAAAAAAAAAAAAAAv3KJ"
-			"cQ=="
+			"cQAAAAAAAP3mxpZuUTQeDggOFhkWDwoOGjFNZ42+4PkAAAAAAAAAAAAAAAAAAAAAAAAAAAAAAAD7"
+			"6cSWcU80HwwKDRYZFw8KCxo0SWiSueL5AAAAAAAAAAAAAADpsXRMR0dRerjr/v3ElFZHR0dHR0dK"
+			"UofI+QAAAAAAAAAAAAAAAAAAAAAAAAAAAAAAAAAAAAAAAAAAAAAAAAAAAAAAAAAAAAAAAAAAAAAA"
+			"AAAAAAAAAAAAAAAAAAAAAAAAAAAAAAAAAAAAAAAAAAAAAAAAAAAAAAAAAAAAAAAAAAAAAAAAAAAA"
+			"AAAAAAAAAAAAAAAAAAAAAAAAAAAAAAAAAAAAAAAAAAAAAAAAAAAAAAAAAAAAAAAAAAAAAAAAAAAA"
+			"AAAAAAAAAAAAAAAAAAAAAAAAAAAAAAAAAAAAAAAAAAAAAAAAAAAAAAAAAAAAAAAAAAAAAAAAAAAA"
+			"AAAAAAAAAAAAAAAAAAAAAAAAAAAAAAAAAAAAAAAAAAAAAAAAAAAAAAAAAAAAAAAAAAAAAAAAAAAA"
+			"AAAAAAAAAAAAAAAAAAAAAAAAAAAAAAAAAAAAAAAAAAAAAAAAAAAAAAAAAAAAAAAAAAAAAAAAAAAA"
+			"AAAAAAAAAAAAAAAAAAAAAAAAAAAAAAAAAAAAAAAAAAAAAAAAAAAAAAAAAAAAAAAAAAAAAAAAAAAA"
+			"AAAAAAAAAAAAAAAAAAAAAAAAAAAAAAAAAAAAAAAAAAAAAAAAAAAAAAAAAAAAAAAAAAAAAAAAAAAA"
+			"AAAAAAAAAAAAAAAAAAAAAAAAAAAAAAAAAAAAAAAAAAAAAAAAAAAAAAAAAAAAAAAAAAAAAAAAAAAA"
+			"AAAAAAAAAAAAAAAAAAAAAAAAAAAAAAAAAAAAAAAAAAAAAAAAAAAAAAAAAAAAAAAAAAAAAAAAAAAA"
+			"AAAAAAAAAAAAAAAAAAAAAAAAAAAAAAAAAAAAAAAAAAAAAAAAAAAAAAAAAAAAAAAAAAAAAAAAAAAA"
+			"AAAAAAAAAAAAAAAAAAAAAAAAAAAAAAAAAAAAAAAAAAAAAAAAAAAAAAAAAAAAAAAAAAAAAAAAAAAA"
+			"AAAAAAAAAAAAAAAAAAAAAAAAAAAAAAAAAAAAAAAAAAAAAAAAAAAAAAAAAAAAAAAAAAAAAAAAAAAA"
+			"AAAAAAAAAAAAAAAAAAAAAAAAAAAAAAAAAAAAAAAAAAAAAAAAAAAAAAAAAAAAAAAAAAAAAAAAAAAA"
+			"AAAAAAAAAAAAAAAAAAAAAAAAAAAAAAAAAAAAAAAAAAAAAAAAAAAAAAAAAAAAAAAAAAAAAAAAAAAA"
+			"AAAAAAAAAAAAAAAAAAAAAAAAAAAAAAAAAAAAAAAAAAAAAAAAAAAAAAAAAAAAAAAAAAAAAAAAAAAA"
+			"AAAAAAAAAAAAAAAAAAAAAAAAAAAAAAAAAAAAAAAAAAAAAAAAAAAAAAAAAAAAAAAAAAAAAAAAAAAA"
+			"AAAAAAAAAAAAAAAAAAAAAAAAAAAAAAAAAAAAAAAAAAAAAAAAAAAAAAAAAAAAAAAAAAAAAAAAAAAA"
+			"AAAAAAAAAAAAAAAAAAAAAAAAAAAAAAAAAAAAAAAAAAAAAAAAAAAAAAAAAAAAAAAAAAAAAAAAAAAA"
+			"AAAAAAAAAAAAAAAAAAAAAAAAAAAAAAAAAAAAAAAAAAAAAAAAAAAAAAAAAAAAAAAAAAAAAAAAAAAA"
+			"AAAAAAAAAAAAAAAAAAAAAAAAAAAAAAAAAAAAAAAAAAAAAAAAAAAAAAAAAAAAAAAAAAAAAAAAAAAA"
+			"AAAAAAAAAAAAAAAAAAAAAAAAAAAAAAAAAAAAAAAAAAAAAAAAAAAAAAAAAAAAAAAAAAAAAAAAAAAA"
+			"AAAAAAAAAAAAAAAAAAAAAAAAAAAAAAAAAAAAAAAAAAAAAAAAAAAAAAAAAAAAAAAAAAAAAAAAAAAA"
+			"AAAAAAAAAAAAAAAAAAAAAAAAAAAAAAAAAAAAAAAAAAAAAAAAAAAAAAAAAAAAAAAAAAAAAAAAAAAA"
+			"AAAAAAAAAAAAAAAAAAAAAAAAAAAAAAAAAAAAAAAAAAAAAAAAAAAAAAAAAAAAAAAAAAAAAAAAAAAA"
+			"AAAAAAAAAAAAAAAAAAAAAAAAAAAAAAAAAAAAAAAAAAAAAAAAAAAAAAAAAAAAAAAAAAAAAAAAAAAA"
+			"AAAAAAAAAAAAAAAAAAAAAAAAAAAAAAAAAAAAAAAAAAAAAAAAAAAAAAAAAAAAAAAAAAAAAAAAAAAA"
+			"AAAAAAAAAAAAAAAAAAAAAAAAAAAAAAAAAAAAAAAAAAAAAAAAAAAAAAAAAAAAAAAAAAAAAAAAAAAA"
+			"AAAAAAAAAAAAAAAAAAAAAAAAAAAAAAAAAAAAAAAAAAAAAAAAAAAAAAAAAAAAAAAAAAAAAAAAAAAA"
+			"AAAAAAAAAAAAAAAAAAAAAAAAAAAAAAAAAAAAAAAAAAAAAAAAAAAAAAAAAAAAAAAAAAAAAAAAAAAA"
+			"AAAAAAAAAAAAAAAAAAAAAAAAAAAAAAAAAAAAAAAAAAAAAAAAAAAAAAAAAAAAAAAAAAAAAAAAAAAA"
+			"AAAAAAAAAAAAAAAAAAAAAAAAAAAAAAAAAAAAAAAAAAAAAAAAAAAAAAAAAAAAAAAAAAAAAAAAAAAA"
+			"AAAAAAAAAAAAAAAAAAAAAAAAAAAAAAAAAAAAAAAAAAAAAAAAAAAAAAAAAAAAAAAAAAAAAAAAAAAA"
+			"AAAAAAAAAAAAAAAAAAAAAAAAAAAAAAAAAAAAAAAAAAAAAAAAAAAAAAAAAAAAAAAAAAAAAAAAAAAA"
+			"AA=="
 		)
 	)

Commit message: Added footprints to resistors and capacitors, and fixed the mosfets wiring issue (#4)
Jul9th push. Added footprints to resistors and capacitors, and fixed the mosfets wiring issue
Parts:
- C13, C14, C21, C3, C4, C8: footprint (none) -> Capacitor_SMD:C_0603_1608Metric
- R10, R11, R12, R14, R19, R20, R23, R24, R27, R41, R6, R7, R8: footprint (none) -> Resistor_SMD:R_0603_1608Metric
Changed lines of the file:
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@@
 			"AAAAAAAAAAAAAAAAAAAAAAAAAAAAAAAAAAAAAAAAAAAAAAAAAAAAAAAAAAAAAAAAAAAAAAAAAAAA"
 			"AAAAAAAAAAAAAAAAAAAAAAAAAAAAAAAAAAAAAAAAAAAAAAAAAAAAAAAAAAAAAAAAAAAAAAAAAAAA"
-			"AA=="
+			"AABFAGkATQBuAHgAdgBQAEcAVQBQAFcAKwA0AHEAagB4AEEAeQA4AC8ASQAwAC8AUAAxAGsAdwBM"
+			"ADMAYQAwAGUANwBTAEMASwBHAGEASgB3ACsAVABlAEQASQBqAG4ARwB5AGEALwBmAGkATwAwAGUA"
+			"bAAwAFQATwBTAGEANgBIAFEANgBhAHAAWQBVAE4ARQBNAEoAVQB0ACsAawBJAGwAawBqAEMANQBQ"
+			"AFcARAB3AFUAKwBrAHIASwAwAE0AbQBiAHcAVQAxAE8AUwBFAFQASgBxAE0AYQBzADIATAB6AEgA"
+			"cwA3AHAAMwBBAHUANwBmADgANwB6ADQAcABsAGgAawA2AHkAQwBZAHQANwBQAFcAbgBtAFkASwAw"
+			"AGwAQgBRACsAMwBjAGoAVQBvAHUAMQBtACsAMgBJAFkAUQBxAEsAcgAzAG8AUwBYAGwAcAB6AEIA"
+			"bwA3AEcAcABuAEoAQwBBAEEATgBIAFoAUABKAG4AYgB3AEUARgAxACsAVABsADUAQQBxAFQAZQA2"
+			"AHIARgBHAHEAegBWACsAcAByAFgASgB4AHQAWQBXAHAASwBXAGsATgBOAEMATgArADQAaAB0AEEA"
+			"WQBRAHgAcgBTAHgATQAwAE0AbgBvAGwASABRACsATQBxAFIAMQBvAE0AVgBZAHoAdAB2AHUAbgBL"
+			"AHEAYwB2AHUAcgBrAGwAagBHADMAOQA1AG8ANAB1ADAAMQB3AGQANQA4ADQAYwBYAFIAZgBEAFIA"
+			"RgAxAG8ASwB0AFoARABGAGIANwBYAE4AVQBBAEEAQQBBAEEAQQBDAEQAOQA2AEgAWgBFAFIAVwBr"
+			"AGwAUwBaAE4AVgBWAEcAcgBuAFQALwBWAEUAUgBVAGsARgBTAGUAdgBUAFoAbgBtAG0AdgBDAEkA"
+			"WABWAFYAVwBVADgAeABGAGkASQBFAFQAcgA2AGUAUwBrAFQAWgA2AEwAaQB5ADQAagBUAFoAVQB3"
+			"AEkAcwB2AFAAOQA3AEgAcQAwAEUAdABEAGwAUgBCAEMAaQBOAFYANwA4AGwAaQB6AFgAZABkAHUA"
+			"QgBsAFcANgB1ADgAcwBpAFEAWABMADAANAB4AEsAYQBoAFoAMgBEAHEATABlADYATwBvAEEAbwBM"
+			"ADYAdABBAFQARwAxAEYAQgBmAEcAeABZAGcAdwBGAEIAUwA2AHEATABTADkAdgBtAGsAUwBXAHgA"
+			"dgArADcAZgA5AC8AUgBpAHcARgBSADIAVgBVAGsAWABiAG0AWAB3ADYAZwBsAEoAeABZAHYAbQA1"
+			"AEsAMgBTAGsAWQBvAC8AUwBBAHEAeQBrAG8AcAAzAEYAaABSADgAWABQAEoAdwBkAGQASABsAEoA"
+			"ZA=="
 		)
 	)
@@
 			"AAAAAAAAAAAAAAAAAAAAAAAAAAAAAAAAAAAAAAAAAAAAAAAAAAAAAAAAAAAAAAAAAAAAAAAAAAAA"
 			"AAAAAAAAAAAAAAAAAAAAAAAAAAAAAAAAAAAAAAAAAAAAAAAAAAAAAAAAAAAAAAAAAAAAAAAAAAAA"
-			"AA=="
+			"AFRmdnY4L0RxL25LZWw0K3h1YmxHOTJKWVhhbW1RdEpidmtMM3ZoSGJaYzMzMkFraGkvczVQeTdQ"
+			"KzhZZTZCZEF5TjNiMzFLMitmVm1oa1lCcVBKQUxBQndteVQyNDVQaml3eFV0Qm5qTjNoSWMyTWJj"
+			"UXBPSUdFbGU0YjIvMHlLT0pDenFjOU15ck91M2N4eHRsRlE3V0E4QTlRVmZFRUFkNVZnNkd0eUpN"
+			"cW5iaTRWOGdWUldRd0VybDFZSWEzc0k4b21ldFk1VVVNZGlXaThCQklZRnVsYldkZHUra0MrVjFI"
+			"QXF2MXdpRTJyZzZnUUE5U0xMZkpiaDFQSE1IWHZyYWpmMzRJbU45TjBEUE4wRFBHZXRLTGl3TlNV"
+			"K2o3RXhVOG9BY3RZRFFMM0JMd0NBT3VJTkhMalp1SFBkWGl1ME03Qkl6YmhkL01waUpqMG1LOHU4"
+			"dGxYemFaL2hOem9NWlRIQVJkOEJ1VU5HMVduN2ZEdDduZFNZakZlM0x5K01pUzAyYjZKWHAvY0VB"
+			"TFlJN0Z5bmZQUlBLU3pLaWRnYWV6MlBJVmxoYk5TenJES0dpRWhzMEdtU1gxZWxsVUxXQTBDOVFU"
+			"RUZVQUMvamdNc1JmNWVRODBTUGg1MStXaGNhZVdKYzJucDNUMW53cFpuZFJqdVZzczM0UWtGUEg0"
+			"ZGY0VHJKVUNkLy9PSkJQN0RQTTBPbnhxMU1qRXVUMTY1L2R6TVBaOGVYSDdYYnZpQU9nOVBBQUIy"
+			"eVhOVFpuZllHUHBsWW53ZUkzOGFQNnZqVDFiNnE1dDRidTRaZW5UQjc1bTFIU2FremdGQVVUaVZE"
+			"OEFHa2MzQ2ZmMUxKMFlNOTQ0a0l4MWpIVjVwVG5FdXo2RFB2TUcvVERCODk4dlZQNERJditPK3pk"
+			"S0pjdzU0THlFamN5MGRYa1ZPVmluUDNuWGU3cjRUSFBBSE00QjZZaDV0djdySHN2UDE4RFp1WWlM"
+			"eVhUYnRkb1Z1dDI4Q1NxNXRpVnk0ejI1eG1JV1NXd2ZyQVVCaCtJWUEyQ0Z5ZFAvcWJMTUZLVS8r"
+			"aU03Tkt1SHBXWnI0dGJkeTBGTmRKMk03Z01CeFVMZXovUU5TYmp5T1RpMHU0WXNzWGF6Yit4bnFZ"
+			"Zm9uQVBVbFQzOVM0aERrNkNKK3A0RGkxUUFBR2tSSlJFRlU4VkREcDZWaDhxRml6eVdlZGttMy9o"
+			"dlJHQUtBd25Ca0FvQWxSVGtSVytNU1RacjBIdVRZeXNNNk1NaGFsYTJVQ3dHS2tsSzI3czh4YWVz"
+			"eXFJdTFSeXY3b0Zab3BRQnFUdURhd3VUaGdiOHVaak5FUk5LOGZmc2ZHOWpxcS9BUUdPc0JRR0g0"
+			"dA=="
 		)
 	)
@@
 			)
 		)
-		(property "Footprint" ""
+		(property "Footprint" "Resistor_SMD:R_0603_1608Metric"
 			(at 24.638 191.77 90)
 			(effects
@@
 			)
 		)
-		(property "Footprint" ""
+		(property "Footprint" "Capacitor_SMD:C_0603_1608Metric"
 			(at 307.0352 149.86 0)
 			(effects
@@
 			)
 		)
-		(property "Footprint" ""
+		(property "Footprint" "Resistor_SMD:R_0603_1608Metric"
 			(at 59.182 82.55 90)
 			(effects
@@
 			)
 		)
-		(property "Footprint" ""
+		(property "Footprint" "Capacitor_SMD:C_0603_1608Metric"
 			(at 36.5252 195.58 0)
 			(effects
@@
 			)
 		)
-		(property "Footprint" ""
+		(property "Footprint" "Resistor_SMD:R_0603_1608Metric"
 			(at 96.012 67.31 90)
 			(effects
@@
 			)
 		)
-		(property "Footprint" ""
+		(property "Footprint" "Resistor_SMD:R_0603_1608Metric"
 			(at 185.42 74.422 90)
 			(effects
@@
 			)
 		)
-		(property "Footprint" ""
+		(property "Footprint" "Resistor_SMD:R_0603_1608Metric"
 			(at 235.458 213.36 90)
 			(effects
@@
 			)
 		)
-		(property "Footprint" ""
+		(property "Footprint" "Resistor_SMD:R_0603_1608Metric"
 			(at 106.172 80.01 90)
 			(effects
@@
 			)
 		)
-		(property "Footprint" ""
+		(property "Footprint" "Resistor_SMD:R_0603_1608Metric"
 			(at 64.008 156.21 90)
 			(effects
@@
 			)
 		)
-		(property "Footprint" ""
+		(property "Footprint" "Resistor_SMD:R_0603_1608Metric"
 			(at 156.21 179.832 90)
 			(effects
@@
 			)
 		)
-		(property "Footprint" ""
+		(property "Footprint" "Resistor_SMD:R_0603_1608Metric"
 			(at 115.062 80.01 90)
 			(effects
@@
 			)
 		)
-		(property "Footprint" ""
+		(property "Footprint" "Capacitor_SMD:C_0603_1608Metric"
 			(at 73.3552 83.82 0)
 			(effects
@@
 			)
 		)
-		(property "Footprint" ""
+		(property "Footprint" "Resistor_SMD:R_0603_1608Metric"
 			(at 235.458 227.33 90)
 			(effects
@@
 			)
 		)
-		(property "Footprint" ""
+		(property "Footprint" "Resistor_SMD:R_0603_1608Metric"
 			(at 190.5 71.882 90)
 			(effects
@@
 			)
 		)
-		(property "Footprint" ""
+		(property "Footprint" "Resistor_SMD:R_0603_1608Metric"
 			(at 21.082 161.29 90)
 			(effects
@@
 			)
 		)
-		(property "Footprint" ""
+		(property "Footprint" "Resistor_SMD:R_0603_1608Metric"
 			(at 156.21 196.342 90)
 			(effects
@@
 			)
 		)
-		(property "Footprint" ""
+		(property "Footprint" "Capacitor_SMD:C_0603_1608Metric"
 			(at 296.8752 149.86 0)
 			(effects
@@
 			)
 		)
-		(property "Footprint" ""
+		(property "Footprint" "Capacitor_SMD:C_0603_1608Metric"
 			(at 98.7552 83.82 0)
 			(effects
@@
 			)
 		)
-		(property "Footprint" ""
+		(property "Footprint" "Capacitor_SMD:C_0603_1608Metric"
 			(at 86.0552 83.82 0)
 			(effects

Commit message: finish schematic
Parts:
- removed SW2, SW3: SW_Push, symbol Switch:SW_Push
- added SW2, SW3: PTS647SN50SMTR2_LFS, custom_footprints:PTS647SK50SMTR2LFS, symbol custom_symbols:PTS647SN50SMTR2_LFS
- C15: renamed from C8; value 10u -> 10uF
- C16: renamed from C21; value 100n -> 100nF
- renumbered C14 to C11, C3 to C12, C4 to C14, Q2 to Q5, Q3 to Q6, R8 to R23, R10 to R24, R14 to R25, R7 to R26, R6 to R27, R23 to R28, R24 to R29, R11 to R30, R12 to R31, R41 to R32, R27 to R33, R19 to R34, R20 to R35, U2 to U4, U1 to U5, U3 to U6
Connections:
- net CHIP_PU: now also SW2.1 (NO_1), SW2.2 (NO_2)
- net GD_SAFE: now also SW3.1 (NO_1), SW3.2 (NO_2); no longer J4.11 (Pin_11), U5.8 (IO9)
- net GND: now also SW2.3 (COM_1), SW2.4 (COM_2), SW3.3 (COM_1), SW3.4 (COM_2)
- net SPI2_CS_GD renamed ~{SPI2_CS}
- new net ~{GD_SAFE}: J4.11 (Pin_11), U5.8 (IO9)
- no-connect marks 21 -> 23
Other:
- note added: "Acceleromter"
- note added: "Address: 0011001b"
- note added: "USB-to-UART Bridge"
- note removed: "Address: 001100xb"
- moved on the sheet: C16
