File: protection.kicad_sch (KiCad schematic)
At the start: 18 parts, among them Q1 SQJQ184ER, Q2 SQJQ184ER, Q3 SQJQ184ER, Q4 SQJQ184ER

Commit message: add manufacturer, mpn, and package to bom
Parts:
- C1: Manufacturer_Name (none) -> Samsung Electro-Mechanics; Manufacturer_Part_Number (none) -> CL10B154KO8NNNC; Package (none) -> 603
- D15: Manufacturer_Name (none) -> Vishay General Semiconductor - Diodes Division; Manufacturer_Part_Number (none) -> VB30100S-E3/8W; Package (none) -> TO263AB
- D5, D8: Manufacturer_Name (none) -> Littelfuse Inc.; Manufacturer_Part_Number (none) -> SMCJ51CA; Package (none) -> DO214AB
- D6: Manufacturer_Name (none) -> STMicroelectronics; Manufacturer_Part_Number (none) -> STPS3L60U; Package (none) -> SMB
- Q1, Q2, Q3, Q4: Manufacturer_Name (none) -> Vishay Siliconix; Manufacturer_Part_Number (none) -> SQJQ184ER-T1_GE3; Package (none) -> PowerPAK 8 x 8
- R10, R11, R5, R7, R8: Manufacturer_Name (none) -> YAGEO; Manufacturer_Part_Number (none) -> RC0603FR-0710RL; Package (none) -> 603
- R12, R13: Manufacturer_Name (none) -> YAGEO; Manufacturer_Part_Number (none) -> AC0603FR-07150KL; Package (none) -> 603
- R14: Manufacturer_Name (none) -> Susumu; Manufacturer_Part_Number (none) -> HRG3216P-1001-D-T1; Package (none) -> 1206
- R6: Manufacturer_Name (none) -> Vishay Dale; Manufacturer_Part_Number (none) -> WSK12161L000FEA; Package (none) -> 1216
